Commit message: tool changeable description

File: mm_description/urdf/mm_tool_changeable.urdf.xacro (robot description, xacro)
@@ -5,5 +5,5 @@
   <xacro:include filename="$(find mm_description)/urdf/mobile_base/swerve_drive.ros2_control.xacro" />
   <xacro:include filename="$(find mm_description)/urdf/mm_sensors.xacro" />
-  <xacro:include filename="$(find mm_description)/urdf/tools/suction_tool.xacro"/>
+  <!-- <xacro:include filename="$(find mm_description)/urdf/tools/suction_tool.xacro"/> -->
   <xacro:arg name="name" default="mm" />
   <xacro:arg name="mobile_type" default="yhs_fw01"/>
@@ -97,9 +97,28 @@
     <origin xyz="0 0 0.06" rpy="0 0 0" />  <!-- position robot on the mobile base -->
   </xacro:ur_robot>
-  <xacro:tool_marco prefix="$(arg arm_prefix)"/>
-  <joint name="$(arg arm_prefix)tool0-tool" type="fixed">
-    <origin xyz="0 0 0" rpy="0 0 0"/>
+  <!-- <xacro:tool_marco prefix="$(arg arm_prefix)"/> -->
+  <link name="$(arg arm_prefix)tool_base"/>
+  <link name="$(arg arm_prefix)pj_tool_tip"/>
+  <link name="$(arg arm_prefix)suction_tool_tip"/>
+  <link name="$(arg arm_prefix)d405_link"/>
+  <joint name="$(arg arm_prefix)tool0-tool_base" type="fixed">
+    <origin xyz="0 0 0" rpy="0 0 -0.78539816339"/>
     <parent link="$(arg arm_prefix)tool0"/>
     <child link="$(arg arm_prefix)tool_base"/>
+  </joint>
+  <joint name="$(arg arm_prefix)pj_tool" type="fixed">
+    <origin xyz="0 -0.041 0.176" rpy="0 0 0"/>
+    <parent link="$(arg arm_prefix)tool_base"/>
+    <child link="$(arg arm_prefix)pj_tool_tip"/>
+  </joint>
+  <joint name="$(arg arm_prefix)suction_tool" type="fixed">
+    <origin xyz="0.02 0 0.33" rpy="0 0 0"/>
+    <parent link="$(arg arm_prefix)tool_base"/>
+    <child link="$(arg arm_prefix)suction_tool_tip"/>
+  </joint>
+  <joint name="$(arg arm_prefix)base-d405" type="fixed">
+    <origin xyz="0.24816342683501683 -0.15421478088509458 -0.09905737640547956" rpy="-1.006184 0.0013119 -1.5359343"/>
+    <parent link="$(arg arm_prefix)base_link"/>
+    <child link="$(arg arm_prefix)d405_link"/>
   </joint>
   <xacro:if value="$(arg sim_gazebo)">

File: mm_moveit_config/srdf/mm_tool_changeable.srdf.xacro (robot description, xacro)
@@ -8,5 +8,5 @@
   <xacro:arg name="arm_type" default="ur"/>
   <xacro:include filename="$(find mm_moveit_config)/srdf/$(arg arm_type)_macro.srdf.xacro"/>
-  <xacro:ur_srdf name="$(arg name)" prefix="$(arg arm_prefix)"/>
+  <xacro:ur_srdf name="$(arg name)" prefix="$(arg arm_prefix)" tool_tip="suction_tool_tip"/>
   <disable_collisions link1="$(arg mobile_prefix)base_link" link2="$(arg arm_prefix)base_link_inertia" reason="Adjacent" />
   <disable_collisions link1="$(arg mobile_prefix)base_link" link2="$(arg mobile_prefix)lf_swerve_link" reason="Adjacent" />

File: mm_moveit_config/srdf/robot.srdf.xacro (robot description, xacro)
@@ -8,5 +8,5 @@
   <xacro:arg name="arm_type" default="ur"/>
   <xacro:include filename="$(find mm_moveit_config)/srdf/$(arg arm_type)_macro.srdf.xacro"/>
-  <xacro:ur_srdf name="$(arg name)" prefix="$(arg arm_prefix)"/>
+  <xacro:ur_srdf name="$(arg name)" prefix="$(arg arm_prefix)" tool_tip="tool_tip"/>
   <disable_collisions link1="$(arg mobile_prefix)base_link" link2="$(arg arm_prefix)base_link_inertia" reason="Adjacent" />
   <disable_collisions link1="$(arg mobile_prefix)base_link" link2="$(arg mobile_prefix)lf_swerve_link" reason="Adjacent" />

File: mm_moveit_config/srdf/ur_macro.srdf.xacro (robot description, xacro)
@@ -5,5 +5,5 @@
     A URDF file must exist for this robot as well, where the joints and the links that are referenced are defined
 -->
-  <xacro:macro name="ur_srdf" params="name prefix">
+  <xacro:macro name="ur_srdf" params="name prefix tool_tip">
     <!--GROUPS - Representation of a set of joints and links. This can be useful for specifying DOF to plan for, defining arms, end effectors, etc-->
     <!--LINKS - When a link is specified, the parent joint of that link (if it exists) is automatically included-->
@@ -11,9 +11,9 @@
     <!--CHAINS - When a chain is specified, all the links along the chain (including endpoints) are included in the group. Additionally, all the joints that are parents to included links are also included. This means that joints along the chain and the parent joint of the base link are included in the group-->
     <!--SUBGROUPS - Groups can also be formed by referencing to already defined group names-->
-    <group name="${prefix}${name}">
-      <chain base_link="${prefix}base_link" tip_link="${prefix}tool_tip" />
+    <group name="${name}">
+      <chain base_link="${prefix}base_link" tip_link="${prefix}${tool_tip}" />
     </group>
     <!--GROUP STATES - Purpose - Define a named state for a particular group, in terms of joint values. This is useful to define states like 'folded arms'-->
-    <group_state name="${prefix}home" group="${prefix}${name}">
+    <group_state name="${prefix}home" group="${name}">
       <joint name="${prefix}elbow_joint" value="0" />
       <joint name="${prefix}shoulder_lift_joint" value="-1.5707" />
@@ -23,5 +23,5 @@
       <joint name="${prefix}wrist_3_joint" value="0" />
     </group_state>
-    <group_state name="${prefix}up" group="${prefix}${name}">
+    <group_state name="${prefix}up" group="${name}">
       <joint name="${prefix}elbow_joint" value="0" />
       <joint name="${prefix}shoulder_lift_joint" value="-1.5707" />
@@ -31,5 +31,5 @@
       <joint name="${prefix}wrist_3_joint" value="0" />
     </group_state>
-    <group_state name="${prefix}test_configuration" group="${prefix}${name}">
+    <group_state name="${prefix}test_configuration" group="${name}">
       <joint name="${prefix}elbow_joint" value="1.4" />
       <joint name="${prefix}shoulder_lift_joint" value="-1.62" />
