Commit message: prepare delta mb model & config

File: mm_description/urdf/mobile_base/wheel.xacro (robot description, xacro)
@@ -137,8 +137,8 @@
         <visual>
             <origin
-                xyz="0 0 0.05"
+                xyz="0 0 0.0125"
                 rpy="0 0 0" />
             <geometry>
-                <box size="0.02 0.02 0.1" />
+                <box size="0.02 0.02 0.025" />
             </geometry>
             <material
