Commit message: iterated load weeled ros control

File: mm_description/urdf/mobile_base/load_swerve_drive.xacro (robot description, xacro)
@@ -52,4 +52,5 @@
     sim_gazebo="$(arg sim_gazebo)"
     use_fake_hardware="$(arg use_fake_hardware)"
+    physical_parameters_file="$(arg physical_parameters_file)"
   />
 </robot>

File: mm_description/urdf/mobile_base/swerve_drive.ros2_control.xacro (robot description, xacro)
@@ -2,5 +2,7 @@
 <robot name="swerve_drive" xmlns:xacro="http://www.ros.org/wiki/xacro">
   <xacro:include filename="$(find mm_description)/urdf/mobile_base/wheel.ros2_control.xacro" />
-  <xacro:macro name="swerve_drive_ros2_control" params="name prefix use_fake_hardware sim_gazebo">
+  <xacro:macro name="swerve_drive_ros2_control" params="name prefix use_fake_hardware sim_gazebo physical_parameters_file">
+    <xacro:property name="config_physical_parameters" value="${xacro.load_yaml(physical_parameters_file)}" />
+    <xacro:property name="wheel_module_list" value="${config_physical_parameters['wheel_module_list']}" />
     <ros2_control name="${name}" type="system">
       <hardware>
@@ -15,8 +17,15 @@
         </xacro:unless>
       </hardware>
-      <xacro:wheel_ros2_control prefix="${prefix}" side="lf_" swerve_id="0" wheel_id="1"/>
-      <xacro:wheel_ros2_control prefix="${prefix}" side="rf_" swerve_id="2" wheel_id="3"/>
-      <xacro:wheel_ros2_control prefix="${prefix}" side="rr_" swerve_id="4" wheel_id="5"/>
-      <xacro:wheel_ros2_control prefix="${prefix}" side="lr_" swerve_id="6" wheel_id="7"/>
+      <xacro:macro name="iterate_include_wheel_module_ros2_control" params="wheel_module_list:=^">
+        <xacro:if value="${wheel_module_list}">
+          <!-- pop first item from list -->
+          <xacro:property name="wheel_module_name" value="${wheel_module_list.pop(0)}"/>
+          <xacro:wheel_ros2_control prefix="${prefix}"
+            side="${wheel_module_name}_" swerve_id="0" wheel_id="1"/>
+          <!-- recursively call myself -->
+          <xacro:iterate_include_wheel_module_ros2_control/>
+        </xacro:if>
+      </xacro:macro>
+      <xacro:iterate_include_wheel_module_ros2_control wheel_module_list="${list(wheel_module_list)}"/>
     </ros2_control>
   </xacro:macro>

Commit message: create and launch mb servo controller

File: mm_description/urdf/mobile_base/load_swerve_drive.xacro (robot description, xacro)
@@ -12,10 +12,10 @@
   <xacro:arg name="physical_parameters_file" default="$(find mm_description)/config/$(arg robot_type)/physical_parameters.yaml" />
   <xacro:arg name="simulation_controllers" default="" />
-  <link name="base_footprint"/>
+  <link name="$(arg prefix)base_footprint"/>
   <xacro:swerve_drive
       name="$(arg name)"
       robot_type="$(arg robot_type)"
       prefix="$(arg prefix)"
-      parent="base_footprint"
+      parent="$(arg prefix)base_footprint"
       geometry_parameters_file="$(arg geometry_parameters_file)"
       physical_parameters_file="$(arg physical_parameters_file)" />
